File: LVJB.kicad_pcb (KiCad board)
At the start: 2 copper layers, 125 x 45 mm, 18 parts, among them J1 Section H1, J10 Section F, J11 Section E1, J12 Section E2, J13 Section E3, J14 Section T1A, J2 Section A1, J3 Section A2, J4 Section A3, J5 Section A4, J6 Section M, J7 Section B1, J8 Section B2, J9 Section K

Commit message: 6 pin conn added for K
Parts:
- J9: footprint Connector_Molex:Molex_Micro-Fit_3.0_43045-1212_2x06_P3.00mm_Vertical -> Connector_Molex:Molex_Micro-Fit_3.0_43045-0612_2x03_P3.00mm_Vertical
- moved J9 4.52 mm to (102.5, 76.0)
Connections:
- H1 pad 1: GND -> (no net)
- H2 pad 1: GND -> (no net)
- H3 pad 1: GND -> (no net)
- H4 pad 1: GND -> (no net)
- J1 pad 7: VCU CAN2 H KH -> VCU CAN2 H EKH
- J1 pad 8: VCU CAN2 L KH -> VCU CAN2 L EKH
- J12 pad 1: VCU CAN2 H EK -> VCU CAN2 H EKH
- J12 pad 9: VCU CAN2 L EK -> VCU CAN2 L EKH
- J9 pad 2: VCU CAN2 H KH -> unconnected-(J9-Pad2)
- J9 pad 3: VCU CAN2 L KH -> VCU Brake 1
- J9 pad 4: unconnected-(J9-Pad4) -> VCU CAN2 H EKH
- J9 pad 5: unconnected-(J9-Pad5) -> VCU CAN2 L EKH
Routing:
- net VCU CAN2 L EKH: track 0.00 -> 43.6 mm
- net VCU CAN2 L EK: track 42.0 -> 0.00 mm
- net VCU CAN2 H EKH: track 0.00 -> 31.8 mm
- net VCU CAN2 H EK: track 20.3 -> 0.00 mm
- net VCU CAN2 L KH: track 7.24 -> 0.00 mm
- net VCU CAN2 H KH: track 7.24 -> 0.00 mm
- net VCU Brake 1: track 44.3 -> 49.8 mm
- net GND: track 547.3 -> 552.0 mm
- net VCU Brake NOT 2: track 31.7 -> 28.9 mm

Commit message: 2mm wiring added
Connections:
- J2 pad 12: Shutdown FA -> GND
- J2 pad 6: GND -> Shutdown FA
- J5 pad 10: GND -> Driven Wheelspeed
- J5 pad 2: BSPD 35kW Test RETURN -> Telemetry CAN H AE
- J5 pad 4: unconnected-(J5-Pad4) -> GND
- J5 pad 7: BSPD 35kW Test IN -> BSPD 35kW Test RETURN
- J5 pad 8: Telemetry CAN H AE -> BSPD 35kW Test IN
- J5 pad 9: Driven Wheelspeed -> unconnected-(J5-Pad9)
Routing:
- net GND: track 552.0 -> 573.8 mm
- net Telemetry CAN H AE: track 25.7 -> 42.0 mm
- net BSPD 35kW Test IN: track 19.0 -> 29.4 mm
- net Driven Wheelspeed: track 72.3 -> 82.5 mm
- net Telemetry CAN L TM: track 99.4 -> 103.3 mm
- net Shutdown FA: track 22.3 -> 26.1 mm
- net Telemetry CAN H TM: track 114.6 -> 118.1 mm
- net Shutdown EF: track 74.2 -> 77.0 mm
- net Shutdown BA: track 50.2 -> 52.0 mm
- net BSPD 35kW Test RETURN: track 19.6 -> 19.0 mm

Commit message: Harness B extra conn added
Connections:
- J7 pad 5: unconnected-(J7-Pad5) -> TSCU Latching Reset
Routing:
- net TSCU Latching Reset: track 15.7 -> 42.1 mm

Commit message: Fixed harness A
Parts:
- moved J14 4.42 mm to (112.5, 71.6)
- moved J9 4.40 mm to (102.5, 71.6)
Connections:
- J13 pad 10: BSPD 35kW Test RETURN -> BSPD 35kW Test IN
- J13 pad 9: BSPD 35kW Test IN -> BSPD 35kW Test RETURN
- J2 pad 11: Ambient Temperature Sensor -> VCU CAN4 H
- J2 pad 12: GND -> VCU Wake
- J2 pad 7: TSAL Safe -> VCU CAN4 L
- J3 pad 12: VCU CAN4 H -> unconnected-(J3-Pad12)
- J3 pad 6: unconnected-(J3-Pad6) -> TSAL Safe
- J3 pad 9: VCU CAN4 L -> unconnected-(J3-Pad9)
- J4 pad 11: VCU Manual Regen Lever -> unconnected-(J4-Pad11)
- J4 pad 7: VCU Wake -> BSPD 35kW Test IN
- J4 pad 8: unconnected-(J4-Pad8) -> BSPD 35kW Test RETURN
- J5 pad 7: BSPD 35kW Test RETURN -> PWM Cooling
- J5 pad 8: BSPD 35kW Test IN -> Tachometer Cooling
Routing:
- net VCU Wake: track 11.5 -> 92.1 mm, vias 0 -> 1
- net VCU Manual Regen Lever: track 38.6 -> 0.00 mm
- net VCU CAN4 H: track 7.20 -> 44.7 mm, vias 0 -> 1
- net BSPD 35kW Test IN: track 29.4 -> 65.4 mm
- net BSPD 35kW Test RETURN: track 19.0 -> 53.3 mm
- net Ambient Temperature Sensor: track 29.4 -> 0.00 mm
- net VCU CAN4 L: track 9.69 -> 38.7 mm, vias 0 -> 1
- net GND: track 573.8 -> 546.5 mm
- net Undriven Wheelspeed: track 56.9 -> 64.9 mm, vias 0 -> 1
- net VCU CAN2 L EKH: track 43.6 -> 50.9 mm
- net Driven Wheelspeed: track 82.5 -> 89.0 mm
- net VCU CAN2 H EKH: track 31.8 -> 38.0 mm, vias 0 -> 1
- net Telemetry CAN L TM: track 103.3 -> 107.9 mm
- net Telemetry CAN H TM: track 118.1 -> 122.6 mm
- net VCU Brake 1: track 49.8 -> 47.5 mm
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
Commit message: Added the 24V pin locations and fixed other issues
Connections:
- J11 pad 10: unconnected-(J11-Pad10) -> J1772 Pilot
- J11 pad 5: TSAL Energized -> unconnected-(J11-Pad5)
- J11 pad 9: unconnected-(J11-Pad9) -> TSAL Energized
- J13 pad 12: J1772 Pilot -> unconnected-(J13-Pad12)
- J2 pad 3: TSAL Energized -> unconnected-(J2-Pad3)
- J3 pad 12: unconnected-(J3-Pad12) -> TSAL Energized
- J7 pad 5: TSCU Latching Reset -> unconnected-(J7-Pad5)
Routing:
- net TSCU Latching Reset: track 42.1 -> 15.7 mm
- net J1772 Pilot: track 35.9 -> 26.6 mm
- net TSAL Energized: track 18.5 -> 14.8 mm

Commit message: added art
Parts:
- added G***: LOGO, LOGO, F.Cu at (106.8, 87.4)
